File: kicad/kicad.kicad_pcb (KiCad board)
At the start: 2 copper layers, 26 parts, among them M1 Fan, M2 Left, M3 Right, Q1 BPW40, Q2 BP103BF, Q3 NPN, U1 PIC16F18875-E/P, U2 L293D, U3 TSSP58038, U4 TSSP58038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

Commit message: components
Parts:
- added J2: headers, Connector_PinHeader_2.54mm:PinHeader_1x05_P2.54mm_Vertical, F.Cu at (75.7, 117.2)
- added J3: Screw_Terminal_01x05, TerminalBlock_Phoenix:TerminalBlock_Phoenix_PT-1,5-5-5.0-H_1x05_P5.00mm_Horizontal, F.Cu at (63.7, 51.2)
- added J4: ~, TerminalBlock_Phoenix:TerminalBlock_Phoenix_PT-1,5-5-5.0-H_1x05_P5.00mm_Horizontal, F.Cu at (63.7, 62.2)
- added SW1: SW_DIP_x01, EZ_TEJ_Library:SW_DIP_SPSTx01_Slide_9.78x4.72mm_W7.62mm_P2.54mm, F.Cu at (80.0, 118.1)
- moved DS1 160.8 mm to (205.5, 101.5)
- moved U1 124.2 mm to (151.2, 49.5)
Connections:
- J1 pad 2: GND -> +12V
- Q1 pad 1: Net-(Q1-C) -> Net-(J4-Pin_1)
- R2 pad 2: Net-(Q1-C) -> Net-(J4-Pin_1)
- U1 pad 19: LMF -> Net-(J3-Pin_4)
- U1 pad 20: LMB -> Net-(J3-Pin_3)
- U1 pad 21: RMF -> Net-(J3-Pin_2)
- U1 pad 22: RMB -> Net-(J3-Pin_1)
- U1 pad 3: Net-(Q1-C) -> Net-(J3-Pin_5)
- U2 pad 10: RMF -> Net-(J4-Pin_3)
- U2 pad 15: RMB -> Net-(J4-Pin_2)
- U2 pad 2: LMF -> Net-(J4-Pin_5)
- U2 pad 7: LMB -> Net-(J4-Pin_4)
Other:
- board outline added: 219.7 x 138.4 mm

Commit message: change pads
Parts:
- J1: footprint EZ_TEJ_Library:TerminalBlock_Phoenix_PT-1,5-3-5.0-H_1x03_P5.00mm_Horizontal -> TerminalBlock_Phoenix:TerminalBlock_Phoenix_PT-1,5-3-5.0-H_1x03_P5.00mm_Horizontal
- J3, J4: footprint TerminalBlock_Phoenix:TerminalBlock_Phoenix_PT-1,5-5-5.0-H_1x05_P5.00mm_Horizontal -> TerminalBlock_Phoenix:TerminalBlock_Phoenix_PT-1,5-8-5.0-H_1x08_P5.00mm_Horizontal
- U2: footprint Package_DIP:DIP-16_W7.62mm -> EZ_TEJ_Library:DIP-16_W7.62mm_LongPads
- moved U5 141.8 mm to (155.3, 40.6), turned to -90 degrees
- moved J1 74.1 mm to (147.3, 40.8), turned to -90 degrees
- moved U1 37.0 mm to (188.0, 45.7)

Commit message: maybe quitting kicad will work
Parts:
- added R7: 1k, EZ_TEJ_Library:R_Axial_DIN0207_L6.3mm_D2.5mm_P7.62mm_Horizontal, F.Cu at (146.1, 111.8)
- Q1, Q2: footprint LED_THT:LED_D5.0mm_Clear -> EZ_TEJ_Library:SolderWire-0.5sqmm_1x02_P4.6mm_D0.9mm_OD2.1mm
- U2: footprint EZ_TEJ_Library:DIP-16_W7.62mm_LongPads -> Package_DIP:DIP-16_W7.62mm
- U3, U4: footprint OptoDevice:Vishay_MINICAST-3Pin -> Connector_Wire:SolderWire-0.5sqmm_1x03_P4.6mm_D0.9mm_OD2.1mm
- moved J2 116.0 mm to (176.5, 59.7)
- moved D2 109.1 mm to (135.9, 109.2), turned to -90 degrees
- moved J3 104.7 mm to (137.2, 125.7)
- moved J4 90.3 mm to (41.9, 149.9)
- moved R1 89.6 mm to (143.5, 64.8)
- moved R4 85.3 mm to (141.0, 85.1)
- moved SW1 78.5 mm to (148.6, 80.0), turned to 180 degrees
- moved RV1 77.8 mm to (182.9, 106.7), turned to 180 degrees
- moved C3 75.4 mm to (142.2, 72.4), turned to 180 degrees
- moved Q2 59.3 mm to (146.1, 88.9), turned to 180 degrees
- moved M1 57.1 mm to (132.1, 109.2), turned to -90 degrees
- moved U4 53.8 mm to (147.3, 100.3), turned to 180 degrees
- moved U3 53.7 mm to (147.3, 92.7), turned to 180 degrees
- moved Q3 49.0 mm to (141.0, 114.3), turned to 90 degrees
- moved U1 38.1 mm to (157.5, 68.6)
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Connections:
- J3 pad 1: Net-(J3-Pin_1) -> GND
- J3 pad 2: Net-(J3-Pin_2) -> +9V
- J3 pad 3: Net-(J3-Pin_3) -> +5V
- J3 pad 6: +5V -> Net-(J3-Pin_6)
- J3 pad 7: +9V -> Net-(J3-Pin_7)
- J3 pad 8: GND -> Net-(J3-Pin_8)
- Q3 pad 2: fan -> Net-(Q3-B)
- U1 pad 11: unconnected-(U1-VDD-Pad11) -> +5V
- U1 pad 12: unconnected-(U1-VSS-Pad12) -> GND
- U1 pad 19: Net-(J3-Pin_4) -> Net-(J3-Pin_5)
- U1 pad 20: Net-(J3-Pin_3) -> Net-(J3-Pin_6)
- U1 pad 21: Net-(J3-Pin_2) -> Net-(J3-Pin_7)
- U1 pad 22: Net-(J3-Pin_1) -> Net-(J3-Pin_8)
- U1 pad 3: Net-(J3-Pin_5) -> Net-(J3-Pin_4)
- U1 pad 31: unconnected-(U1-VSS-Pad31) -> GND
- U1 pad 32: unconnected-(U1-VDD-Pad32) -> +5V
Routing:
- net GND: track 0.00 -> 325.3 mm
- net +5V: track 0.00 -> 260.8 mm
- net +9V: track 0.00 -> 97.3 mm
- net Net-(J3-Pin_4): track 0.00 -> 73.3 mm
- net +12V: track 0.00 -> 54.3 mm
- net Net-(J2-Pin_1): track 0.00 -> 47.3 mm
- net fan: track 0.00 -> 28.4 mm
- net Net-(U1-RA4): track 0.00 -> 24.2 mm
- net Net-(DS1-VO): track 0.00 -> 19.4 mm
- net Net-(U1-RA3): track 0.00 -> 19.0 mm
- net Net-(Q2-C): track 0.00 -> 18.9 mm
- net Net-(DS1-D6): track 0.00 -> 15.3 mm
- net Net-(DS1-D4): track 0.00 -> 15.3 mm
- net Net-(DS1-D5): track 0.00 -> 15.3 mm
- net Net-(DS1-D7): track 0.00 -> 15.3 mm
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Other:
- board size 219.7 x 138.4 mm -> 165.1 x 124.5 mm

Commit message: scheduling system
Parts:
- J1: footprint TerminalBlock_Phoenix:TerminalBlock_Phoenix_PT-1,5-3-5.0-H_1x03_P5.00mm_Horizontal -> EZ_TEJ_Library:TerminalBlock_Phoenix_PT-1,5-3-5.0-H_1x03_P5.00mm_Horizontal
- moved DS1 2.54 mm to (188.0, 95.2)
- moved J2 2.54 mm to (179.1, 59.7)
Routing:
- net GND: track 325.3 -> 330.9 mm
- net +5V: track 260.8 -> 266.2 mm
- net Net-(DS1-D6): track 15.3 -> 17.9 mm
- net Net-(DS1-D7): track 15.3 -> 17.9 mm
- net Net-(DS1-R/W): track 13.2 -> 15.8 mm
- net Net-(DS1-RS): track 13.2 -> 15.8 mm
- net Net-(DS1-E): track 13.2 -> 15.8 mm
- net Net-(DS1-D5): track 15.3 -> 17.9 mm
- net Net-(DS1-D4): track 15.3 -> 17.9 mm
- net Net-(J2-Pin_1): track 47.3 -> 49.3 mm
- net Net-(J3-Pin_5): track 13.5 -> 15.0 mm
- net Net-(DS1-VO): track 19.4 -> 20.9 mm
Other:
- board size 165.1 x 124.5 mm -> 166.4 x 124.5 mm
